File: hardware/eurorack-pmod-pcb-flat/eurorack-pmod-panel/eurorack-pmod-panel.kicad_pcb (KiCad board)
At the start: 2 copper layers, 15 x 128.5 mm, 11 parts

Commit message: rev2-flat: front panel fab1
Other:
- board text added: "VK2 SEB"
- board text added: "α"
- board text added: "β"
- board text added: "γ"
- board text added: "δ"
- board text removed: "VK2SEB"
