File: hardware/eurorack-pmod-r3/dual_mono_outputs.kicad_sch (KiCad schematic)
At the start: 14 parts, among them J8 PJ-324M0, J9 PJ-324M0, U2 TL074

Commit message: rev3/pcb: preliminary fab outputs and text labels
Parts:
- J8, J9: value PJ-324M0 -> AUDIO JACK PJ-324M0
- U2: value TL074 -> TL074 OP AMP
Changed lines of the file:
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@@
     (in_bom yes) (on_board yes)
     (property "Reference" "J8" (id 0) (at 104.14 34.925 0))
-    (property "Value" "PJ-324M0" (id 1) (at 104.14 37.465 0))
+    (property "Value" "AUDIO JACK PJ-324M0" (id 1) (at 104.14 37.465 0))
     (property "Footprint" "AudioJacksFixed:pj324m" (id 2) (at 104.14 40.64 0)
       (effects (font (size 1.27 1.27)) hide)
@@
     (in_bom yes) (on_board yes)
     (property "Reference" "J9" (id 0) (at 102.87 92.075 0))
-    (property "Value" "PJ-324M0" (id 1) (at 102.87 94.615 0))
+    (property "Value" "AUDIO JACK PJ-324M0" (id 1) (at 102.87 94.615 0))
     (property "Footprint" "AudioJacksFixed:pj324m" (id 2) (at 102.87 97.79 0)
       (effects (font (size 1.27 1.27)) hide)
@@
     (in_bom yes) (on_board yes) (fields_autoplaced)
     (property "Reference" "U2" (id 0) (at 54.61 92.329 0))
-    (property "Value" "TL074" (id 1) (at 54.61 94.869 0))
+    (property "Value" "TL074 OP AMP" (id 1) (at 54.61 94.869 0))
     (property "Footprint" "Package_SO:SOIC-14_3.9x8.7mm_P1.27mm" (id 2) (at 53.34 100.33 0)
       (effects (font (size 1.27 1.27)) hide)
@@
     (in_bom yes) (on_board yes) (fields_autoplaced)
     (property "Reference" "U2" (id 0) (at 49.53 35.56 0))
-    (property "Value" "TL074" (id 1) (at 49.53 38.1 0))
+    (property "Value" "TL074 OP AMP" (id 1) (at 49.53 38.1 0))
     (property "Footprint" "Package_SO:SOIC-14_3.9x8.7mm_P1.27mm" (id 2) (at 48.26 43.18 0)
       (effects (font (size 1.27 1.27)) hide)

Commit message: try routing with capsense groundfix
Parts:
- added Q? (x2): 2N7002E, Package_TO_SOT_SMD:SOT-23, symbol Transistor_FET:2N7002E
- added R34 (x2): 4K7, Resistor_SMD:R_0402_1005Metric, symbol Device:R
Connections:
- net GND: now also Q?.2 (S), Q?.2 (S); no longer J8.G, J9.G
- net JACK_DETECT1: now also R34.2
- net JACK_DETECT2: now also R34.2
- net TIP_NO1: now reaches J8.TN
- net TIP_NO2: now reaches J9.TN
- new net: Q?.1 (G), R34.1 (x2)
- new net CAP_SENSE1: J8.G, Q?.3 (D)
- new net CAP_SENSE2: J9.G, Q?.3 (D)
- no-connect marks 2 -> 0
Other:
- moved on the sheet: R18, R22
