File: hardware/eurorack-pmod-r3/dual_mono_outputs.kicad_sch (KiCad schematic)
At the start: 18 parts, among them J8 AUDIO JACK PJ-324M0, J9 AUDIO JACK PJ-324M0, U2 TL074 OP AMP

Commit message: fab: add gerber/pnp for r3.2 sent 3 Oct 23
Parts:
- removed Q? (x2): 2N7002E, Package_TO_SOT_SMD:SOT-23, symbol Transistor_FET:2N7002E
- removed R34 (x2): 4K7, Resistor_SMD:R_0402_1005Metric, symbol Device:R
