File: hardware/eurorack-pmod-r3.3/eurorack-pmod-pcb.kicad_sch (KiCad schematic)
At the start: 24 parts, among them Q1 2N7002E, U1 AK4619VN AUDIO CODEC, U2 TL074 OP AMP, U3 TL074 OP AMP, U4 PCA9557PW IO EXPANDER, U5 24AA025UIDT EEPROM, U6 CY8CMBR3108

Commit message: hardware/fab: push latest from 25.11.23 batch (#55)
* Swap FFC for CTXJ-H2.0. Pinswap capsense OUT1-4 reverse
* Convert BOM/CPL
* Add gerbers sent 25 Nov
Connections:
- net at RN8.1 (R1.1): now also U6.10 (CS6); no longer U6.9 (CS5)
- net at RN8.1 (R1.1): now also U6.8 (CS4); no longer U6.11 (CS7)
- net at RN8.1 (R1.1): now also U6.11 (CS7); no longer U6.8 (CS4)
- net at RN8.1 (R1.1): now also U6.9 (CS5); no longer U6.10 (CS6)
Other:
- moved on the sheet: RN8A
