File: hardware/eurorack-pmod-r3.3/power_conn.kicad_sch (KiCad schematic)
At the start: 23 parts, among them J1 CONN 2x5 P=2.54mm, J2 CONN 2x6 P=2.54mm, J3 Conn_01x14_Socket

Commit message: hardware/fab: push latest from 25.11.23 batch (#55)
* Swap FFC for CTXJ-H2.0. Pinswap capsense OUT1-4 reverse
* Convert BOM/CPL
* Add gerbers sent 25 Nov
Parts:
- J3: footprint Connector_FFC-FPC:Hirose_FH12-14S-0.5SH_1x14-1MP_P0.50mm_Horizontal -> ffc-ctxj:FFC_0.5-14P_CTXJ-H2.0_1; lcsc# C5378715 -> C5373472
Changed lines of the file:
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@@
       (effects (font (size 1.27 1.27)) (justify left))
     )
-    (property "Footprint" "Connector_FFC-FPC:Hirose_FH12-14S-0.5SH_1x14-1MP_P0.50mm_Horizontal" (at 153.924 53.848 0)
+    (property "Footprint" "ffc-ctxj:FFC_0.5-14P_CTXJ-H2.0_1" (at 153.924 53.848 0)
       (effects (font (size 1.27 1.27)) hide)
     )
@@
       (effects (font (size 1.27 1.27)) hide)
     )
-    (property "lcsc#" "C5378715" (at 153.924 53.848 0)
+    (property "lcsc#" "C5373472" (at 153.924 53.848 0)
       (effects (font (size 1.27 1.27)) hide)
     )
